File: Balancer.kicad_sch (KiCad schematic)
At the start: 23 parts, among them J4 Balance, J5 Conn_01x06, SW5 Reset, SW6 Button, U17 LDO_Diodes_AP7370, U6 74HC4051, U7 74HC4051, U8 Module_NINA-B306

Commit message: stream 24-01-10
Parts:
- removed C12: 100n, Capacitor_SMD:C_0402_1005Metric, symbol Device:C
Changed lines of the file:
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@@
   (junction (at 142.24 143.51) (diameter 0) (color 0 0 0 0)
-  )
-  (wire (pts (xy 198.12 49.53) (xy 198.12 60.96))
-    (stroke (width 0) (type default) (color 0 0 0 0))
   )
   (wire (pts (xy 251.46 116.84) (xy 251.46 118.11))
@@
     )
     (property "Datasheet" "~" (id 3) (at 227.33 134.62 0)
-      (effects (font (size 1.27 1.27)) hide)
-    )
-    (pin "1")
-    (pin "2")
-  )
-  (symbol (lib_id "Device:C") (at 198.12 45.72 0) (unit 1)
-    (in_bom yes) (on_board yes) (fields_autoplaced)
-    (property "Reference" "C12" (id 0) (at 201.93 44.4499 0)
-      (effects (font (size 1.27 1.27)) (justify left))
-    )
-    (property "Value" "100n" (id 1) (at 201.93 46.9899 0)
-      (effects (font (size 1.27 1.27)) (justify left))
-    )
-    (property "Footprint" "Capacitor_SMD:C_0402_1005Metric" (id 2) (at 199.0852 49.53 0)
-      (effects (font (size 1.27 1.27)) hide)
-    )
-    (property "Datasheet" "~" (id 3) (at 198.12 45.72 0)
       (effects (font (size 1.27 1.27)) hide)
     )
@@
     (pin "2")
   )
-  (symbol (lib_id "power:GND") (at 198.12 60.96 0) (unit 1)
-    (in_bom yes) (on_board yes) (fields_autoplaced)
-    (property "Reference" "#PWR040" (id 0) (at 198.12 67.31 0)
-      (effects (font (size 1.27 1.27)) hide)
-    )
-    (property "Value" "GND" (id 1) (at 198.247 65.3542 0)
-      (effects (font (size 1.27 1.27)) hide)
-    )
-    (property "Footprint" "" (id 2) (at 198.12 60.96 0)
-      (effects (font (size 1.27 1.27)) hide)
-    )
-    (property "Datasheet" "" (id 3) (at 198.12 60.96 0)
-      (effects (font (size 1.27 1.27)) hide)
-    )
-    (pin "1")
-  )
   (symbol (lib_id "power:GND") (at 134.62 60.96 0) (unit 1)
