File: 8-Cell Balancer Charger.kicad_pcb (KiCad board)
At the start: 2 copper layers, 60 x 60 mm, 242 parts, among them J4 Balance, J5 Conn_01x06, Q1 Q_NMOS_DGS, Q10 BSS84AKW, Q11 BSS84AKW, Q12 PMXB360ENEA, Q13 2SA1832, Q14 IRLU120NPBF, Q15 BSS84AKW, Q16 BSS84AKW, Q17 PMXB360ENEA, Q18 2SA1832, Q19 IRLU120NPBF, Q2 Q_PMOS_DGS, Q20 BSS84AKW, Q21 BSS84AKW, Q22 PMXB360ENEA, Q23 2SA1832, Q24 IRLU120NPBF, Q25 BSS84AKW, Q26 BSS84AKW, Q27 PMXB360ENEA, Q28 2SA1832, Q29 IRLU120NPBF, Q3 Q_NMOS_DGS, Q30 BSS84AKW, Q31 BSS84AKW, Q32 PMXB360ENEA, Q33 2SA1832, Q34 IRLU120NPBF, Q35 BSS84AKW, Q36 BSS84AKW, Q37 PMXB360ENEA, Q38 2SA1832, Q39 IRLU120NPBF, Q4 Q_NMOS_DGS, Q40 BSS84AKW, Q41 BSS84AKW, Q42 PMXB360ENEA, Q43 2SA1832, Q44 IRLU120NPBF, Q45 BSS84AKW, Q46 BSS84AKW, Q5 Q_NMOS_DGS, Q6 Q_NMOS_DGS, Q7 PMXB360ENEA, Q8 2SA1832, Q9 IRLU120NPBF, SW5 Reset, SW6 Button, U1 FAN3278, U10 TLV9052, U11 TLV9052, U12 TLV9052, U13 TLV9052, U14 TLV9052, U15 TLV9052, U16 TLV9052, U17 LDO_Diodes_AP7370, U3 ATmega4809-A, U6 74HC4051, U7 74HC4051, U8 Module_NINA-B306, U9 TLV9052

Commit message: stream 24-01-10
Parts:
- removed C12: 100n, Capacitor_SMD:C_0402_1005Metric
- removed G***: LOGO, 0_ProjectLibrary:jb_6mm
- added C41: 100n, Capacitor_SMD:C_0402_1005Metric, F.Cu at (35.7, 94.0)
- added C42: 100n, Capacitor_SMD:C_0402_1005Metric, F.Cu at (35.8, 91.4)
- added C43: 100n, Capacitor_SMD:C_0402_1005Metric, F.Cu at (50.4, 87.0)
- added C44: 100n, Capacitor_SMD:C_0402_1005Metric, F.Cu at (47.6, 87.0)
- added C45: 100n, Capacitor_SMD:C_0402_1005Metric, F.Cu at (41.0, 93.6)
- added C46: 100n, Capacitor_SMD:C_0402_1005Metric, F.Cu at (38.1, 93.6)
- added C47: 100n, Capacitor_SMD:C_0402_1005Metric, F.Cu at (31.6, 100.2)
- added C48: 100n, Capacitor_SMD:C_0402_1005Metric, F.Cu at (28.7, 100.2)
- added C49: 100n, Capacitor_SMD:C_0402_1005Metric, F.Cu at (41.0, 87.0)
- added C50: 100n, Capacitor_SMD:C_0402_1005Metric, F.Cu at (38.1, 87.0)
- added C51: 100n, Capacitor_SMD:C_0402_1005Metric, F.Cu at (31.6, 93.6)
- added C52: 100n, Capacitor_SMD:C_0402_1005Metric, F.Cu at (28.7, 93.6)
- added C53: 100n, Capacitor_SMD:C_0402_1005Metric, F.Cu at (31.6, 87.0)
- added C54: 100n, Capacitor_SMD:C_0402_1005Metric, F.Cu at (28.7, 87.0)
- added C55: 100n, Capacitor_SMD:C_0402_1005Metric, F.Cu at (50.4, 93.6)
- added C56: 100n, Capacitor_SMD:C_0402_1005Metric, F.Cu at (47.6, 93.6)
- added REF**: DFN-8-1EP_2x2mm_P0.5mm_EP0.6x1.2mm, Package_DFN_QFN:DFN-8-1EP_2x2mm_P0.5mm_EP0.6x1.2mm, F.Cu at (107.6, 54.3)
- added REF**: SOT-23-8, Package_TO_SOT_SMD:SOT-23-8, F.Cu at (101.5, 54.6)
- added U9: TLV9052, Package_SO:MSOP-8_3x3mm_P0.65mm, F.Cu at (101.9, 59.4)
- U10, U11, U12, U13, U14, U15, U16, U9: footprint Package_SO:MSOP-8_3x3mm_P0.65mm -> Package_TO_SOT_SMD:SOT-23-8
- moved R36 47.9 mm to (149.6, 61.6), turned to -90 degrees
- moved Q9 39.2 mm to (143.4, 62.5), turned to 90 degrees
- moved C17 36.0 mm to (138.0, 65.9), turned to 0 degrees
- moved R37 32.3 mm to (138.5, 63.4), turned to 90 degrees
- moved R35 32.0 mm to (138.5, 61.5), turned to -90 degrees
- moved R41 31.9 mm to (137.1, 59.3), turned to 180 degrees
- moved R38 31.8 mm to (138.0, 64.9), turned to 0 degrees
- moved C16 31.0 mm to (133.9, 62.4)
- moved C15 30.5 mm to (138.5, 59.6), turned to -90 degrees
- moved R34 30.1 mm to (135.3, 59.3), turned to 0 degrees
- moved U9 28.5 mm to (136.2, 62.3), turned to 90 degrees
- moved R39 27.2 mm to (135.5, 64.9)
- moved R33 24.0 mm to (135.5, 65.9), turned to 180 degrees
- moved Q10 23.6 mm to (132.7, 65.0), turned to 180 degrees
- moved Q11 22.6 mm to (132.7, 60.0), turned to 180 degrees
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Routing:
- net /Balancer/Balancer3/Cell+: track 149.2 -> 118.0 mm, vias 39 -> 27
- net /Balancer/Balancer5/Cell+: track 149.2 -> 121.0 mm, vias 39 -> 30
- net /Balancer/Balancer2/Cell+: track 128.3 -> 112.9 mm, vias 36 -> 33
- net Net-(Q30-Pad2): track 18.0 -> 33.4 mm, vias 0 -> 3
- net Net-(Q15-Pad2): track 18.0 -> 33.4 mm, vias 0 -> 3
- net Net-(Q40-Pad2): track 18.0 -> 33.4 mm, vias 0 -> 3
- net Net-(Q35-Pad2): track 18.0 -> 33.4 mm, vias 0 -> 3
- net Net-(Q25-Pad2): track 18.0 -> 33.4 mm, vias 0 -> 3
- net Net-(Q20-Pad2): track 18.0 -> 33.4 mm, vias 0 -> 3
- net /Balancer/Supply: track 166.6 -> 154.2 mm
- net /Balancer/Balancer1/Cell+: track 77.7 -> 65.3 mm
- net Net-(C30-Pad1): track 38.6 -> 48.4 mm, vias 0 -> 3
- net Net-(C24-Pad1): track 38.6 -> 48.4 mm, vias 0 -> 3
- net /Balancer/Balancer6/Cell+: track 115.5 -> 106.1 mm, vias 30 -> 33
- net Net-(Q45-Pad2): track 12.0 -> 17.1 mm, vias 0 -> 1
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
Commit message: Update
Parts:
- removed the REF** at (107.6, 54.3)
- removed the REF** at (101.5, 54.6)
- removed the U9 at (101.9, 59.4)
- added NT1: NetTie_2, 0_ProjectLibrary:NetTie-2_SMD_Pad0.127mm, F.Cu at (115.8, 95.2)
- added NT2: NetTie_2, 0_ProjectLibrary:NetTie-2_SMD_Pad0.127mm, F.Cu at (107.8, 95.2)
- added NT3: NetTie_2, 0_ProjectLibrary:NetTie-2_SMD_Pad0.127mm, F.Cu at (99.8, 95.2)
- added NT4: NetTie_2, 0_ProjectLibrary:NetTie-2_SMD_Pad0.127mm, F.Cu at (91.8, 95.2)
- added NT5: NetTie_2, 0_ProjectLibrary:NetTie-2_SMD_Pad0.127mm, F.Cu at (89.2, 104.8)
- added NT6: NetTie_2, 0_ProjectLibrary:NetTie-2_SMD_Pad0.127mm, F.Cu at (97.2, 104.8)
- added NT7: NetTie_2, 0_ProjectLibrary:NetTie-2_SMD_Pad0.127mm, F.Cu at (105.2, 104.8)
- added NT8: NetTie_2, 0_ProjectLibrary:NetTie-2_SMD_Pad0.127mm, F.Cu at (113.2, 104.8)
- moved C54 60.0 mm to (84.4, 109.3), turned to 180 degrees
- moved C38 58.7 mm to (117.9, 116.4), turned to 90 degrees
- moved C52 58.2 mm to (84.4, 110.3), turned to 180 degrees
- moved C48 56.4 mm to (84.4, 91.7), turned to 180 degrees
- moved C50 52.3 mm to (84.4, 111.3), turned to 180 degrees
- moved C42 48.7 mm to (84.4, 88.7), turned to 180 degrees
- moved R36 47.9 mm to (115.4, 95.2), turned to 180 degrees
- moved C53 47.6 mm to (73.6, 109.3)
- moved C46 46.4 mm to (84.4, 90.7), turned to 180 degrees
- moved C51 45.2 mm to (73.6, 110.3)
- moved C47 42.9 mm to (73.6, 91.7)
- moved C49 40.7 mm to (73.6, 111.3)
- moved C56 39.7 mm to (84.4, 108.3), turned to 180 degrees
- moved Q9 39.2 mm to (114.5, 89.0), turned to 0 degrees
- moved C41 38.3 mm to (73.6, 88.7), turned to 0 degrees
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Connections:
- R106 pad 1: /Balancer/Balancer3/Cell+ -> Net-(NT6-Pad2)
- R119 pad 1: /Balancer/Balancer2/Cell+ -> Net-(NT7-Pad2)
- R132 pad 1: /Balancer/Balancer1/Cell+ -> Net-(NT8-Pad2)
- R41 pad 1: /Balancer/Balancer8/Cell+ -> Net-(NT1-Pad2)
- R54 pad 1: /Balancer/Balancer7/Cell+ -> Net-(NT2-Pad2)
- R67 pad 1: /Balancer/Balancer6/Cell+ -> Net-(NT3-Pad2)
- R80 pad 1: /Balancer/Balancer5/Cell+ -> Net-(NT4-Pad2)
- R93 pad 1: /Balancer/Supply -> Net-(NT5-Pad2)
Routing:
- net /Balancer/Supply: track 154.2 -> 95.8 mm, vias 33 -> 13
- net /Balancer/Balancer2/Cell+: track 112.9 -> 54.5 mm, vias 33 -> 13
- net /Balancer/Balancer6/Cell+: track 106.1 -> 54.5 mm, vias 33 -> 13
- net /Balancer/Balancer5/Cell+: track 121.0 -> 72.4 mm, vias 30 -> 13
- net /Balancer/Balancer7/Cell+: track 85.2 -> 36.9 mm, vias 20 -> 13
- net /Balancer/Balancer3/Cell+: track 118.0 -> 72.4 mm, vias 27 -> 13
- net Net-(Q34-Pad2): track 52.9 -> 15.3 mm
- net Net-(Q39-Pad2): track 52.9 -> 15.3 mm
- net Net-(Q29-Pad2): track 52.9 -> 15.3 mm
- net Net-(Q24-Pad2): track 52.9 -> 15.3 mm
- net Net-(Q19-Pad2): track 52.9 -> 15.3 mm
- net Net-(Q14-Pad2): track 52.9 -> 15.3 mm
- net Net-(C30-Pad1): track 48.4 -> 15.6 mm, vias 3 -> 0
- net Net-(C24-Pad1): track 48.4 -> 15.6 mm, vias 3 -> 0
- net Net-(C21-Pad1): track 48.4 -> 15.6 mm, vias 3 -> 0
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Other:
- board size 60 x 60 mm -> 60 x 50 mm

Commit message: stream 24-01-24
Parts:
- added G***: LOGO, 0_ProjectLibrary:jb_6mm, F.Cu at (68.9, 109.0)
- moved R18 118.3 mm to (149.3, 121.5)
- moved R12 113.9 mm to (163.6, 114.2)
- moved C6 102.0 mm to (174.5, 112.2)
- moved C4 94.2 mm to (177.4, 112.2)
- moved R17 65.9 mm to (158.0, 118.2)
- moved R19 65.8 mm to (153.8, 116.1)
- moved C3 64.6 mm to (163.1, 116.2)
- moved R11 60.4 mm to (152.2, 121.5)
- moved R4 56.8 mm to (155.1, 120.4)
- moved R13 54.8 mm to (146.4, 123.6)
- moved R2 53.8 mm to (155.1, 122.4)
- moved C2 49.9 mm to (165.9, 116.2)
- moved R8 47.8 mm to (152.2, 123.5)
- moved R14 47.4 mm to (219.0, 84.5)
- moved R15 46.7 mm to (228.0, 74.7)
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Routing:
- net +3.3V: track 56.6 -> 76.8 mm, vias 4 -> 3
- net /Balancer/Balancer8/Cell+: track 13.3 -> 27.6 mm
- net /Balancer/Balancer1/Cell+: track 36.9 -> 46.4 mm
- net /Balancer/Balancer7/Cell+: track 36.9 -> 46.4 mm
- net /Balancer/BUTTON: track 4.12 -> 9.21 mm
- net /Balancer/Balancer6/Cell+: track 54.5 -> 59.2 mm
- net /Balancer/Balancer2/Cell+: track 54.5 -> 59.0 mm
- net GND: track 7.84 -> 11.2 mm, vias 36 -> 43
- net /Balancer/CurrentCell8: track 50.7 -> 54.0 mm
- net /Balancer/VoltageCell8: track 50.3 -> 53.4 mm
- net /Balancer/CurrentCell4: track 23.4 -> 26.5 mm
- net /Balancer/VoltageCell4: track 29.9 -> 33.0 mm
- net /Balancer/VoltageCell6: track 34.3 -> 37.3 mm
- net /Balancer/VoltageCell2: track 48.4 -> 51.5 mm
- net /Balancer/CurrentCell6: track 36.7 -> 39.8 mm
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Other:
- board text added: "8-Cell Balancer by jbussmann"
