File: 8-Cell Balancer.kicad_sch (KiCad schematic)
At the start: 24 parts, among them J1 Balance, J2 Conn_01x06, SW1 Reset, SW2 Button, U1 AP7370, U2 74HC4051, U3 74HC4051, U4 NINA-B306

Commit message: finalize component values
Parts:
- J2: value Conn_01x06 -> SWD
- R1, R2: value 51k -> 47k
- R3, R4, R5: value 1.8k -> 620R
Other:
- note added: "Improvements: - BJT instead of FET (price/rail margin) - switching level shifter - Footprint RGB-LED"
