File: Blancer1-8.kicad_sch (KiCad schematic)
At the start: 23 parts, among them Q10 BSS84AKW, Q11 BSS84AKW, Q7 PMXB360ENEA, Q8 2SA1832, Q9 IRLU120NPBF, U9 TLV9052

Commit message: stream 24-01-10
Parts:
- added C41, C42: 100n, Capacitor_SMD:C_0402_1005Metric, symbol Device:C
- U9: footprint Package_SO:MSOP-8_3x3mm_P0.65mm -> Package_TO_SOT_SMD:SOT-23-8
Connections:
- net BalaceCurrent: now also C42.1
- net CellVoltage: now also C41.1
- net GND: now also C41.2, C42.2
Other:
- note added: "tau = 1/(2*pi*f_{c}) = 1/(ω_{c}) R*C = 100k*100n = 10ms -> 16Hz R*C = 100k*1u = 100ms -> 1.6Hz"
Changed lines of the file:
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@@
   (junction (at 181.61 127) (diameter 0) (color 0 0 0 0)
   )
+  (junction (at 191.77 71.12) (diameter 0) (color 0 0 0 0)
+  )
+  (junction (at 191.77 127) (diameter 0) (color 0 0 0 0)
+  )
   (junction (at 146.05 67.31) (diameter 0) (color 0 0 0 0)
   )
@@
     (stroke (width 0) (type default) (color 0 0 0 0))
   )
+  (wire (pts (xy 191.77 71.12) (xy 194.31 71.12))
+    (stroke (width 0) (type default) (color 0 0 0 0))
+  )
   (wire (pts (xy 181.61 113.03) (xy 181.61 114.3))
     (stroke (width 0) (type default) (color 0 0 0 0))
@@
     (stroke (width 0) (type default) (color 0 0 0 0))
   )
+  (wire (pts (xy 191.77 127) (xy 194.31 127))
+    (stroke (width 0) (type default) (color 0 0 0 0))
+  )
   (wire (pts (xy 129.54 48.26) (xy 134.62 48.26))
     (stroke (width 0) (type default) (color 0 0 0 0))
@@
     (stroke (width 0) (type default) (color 0 0 0 0))
   )
-  (wire (pts (xy 181.61 127) (xy 182.88 127))
+  (wire (pts (xy 181.61 127) (xy 191.77 127))
     (stroke (width 0) (type default) (color 0 0 0 0))
   )
@@
     (stroke (width 0) (type default) (color 0 0 0 0))
   )
+  (wire (pts (xy 191.77 135.89) (xy 191.77 137.16))
+    (stroke (width 0) (type default) (color 0 0 0 0))
+  )
   (wire (pts (xy 156.21 118.11) (xy 156.21 114.3))
     (stroke (width 0) (type default) (color 0 0 0 0))
@@
     (stroke (width 0) (type default) (color 0 0 0 0))
   )
+  (wire (pts (xy 191.77 71.12) (xy 191.77 72.39))
+    (stroke (width 0) (type default) (color 0 0 0 0))
+  )
+  (wire (pts (xy 191.77 127) (xy 191.77 128.27))
+    (stroke (width 0) (type default) (color 0 0 0 0))
+  )
   (wire (pts (xy 156.21 114.3) (xy 181.61 114.3))
     (stroke (width 0) (type default) (color 0 0 0 0))
@@
     (stroke (width 0) (type default) (color 0 0 0 0))
   )
-  (wire (pts (xy 181.61 71.12) (xy 182.88 71.12))
+  (wire (pts (xy 181.61 71.12) (xy 191.77 71.12))
     (stroke (width 0) (type default) (color 0 0 0 0))
   )
@@
     (stroke (width 0) (type default) (color 0 0 0 0))
   )
+  (wire (pts (xy 191.77 80.01) (xy 191.77 81.28))
+    (stroke (width 0) (type default) (color 0 0 0 0))
+  )
   (wire (pts (xy 172.72 120.65) (xy 173.99 120.65))
     (stroke (width 0) (type default) (color 0 0 0 0))
@@
     (stroke (width 0) (type default) (color 0 0 0 0))
   )
-  (text "Pmax = 33V * 10uA = 330uW" (at 199.39 121.92 0)
+  (text "Pmax = 33V * 10uA = 330uW" (at 199.39 119.38 0)
     (effects (font (size 1.27 1.27)) (justify left bottom))
   )
@@
     (effects (font (size 1.27 1.27)) (justify left bottom))
   )
-  (text "Vgs margin to rail\n-3.1...-4.4V @ 10uA" (at 199.39 118.11 0)
-    (effects (font (size 1.27 1.27)) (justify left bottom))
-  )
-  (text "I_{leakage} = 1uA" (at 200.66 127 0)
+  (text "Vgs margin to rail\n-3.1...-4.4V @ 10uA" (at 199.39 115.57 0)
+    (effects (font (size 1.27 1.27)) (justify left bottom))
+  )
+  (text "I_{leakage} = 1uA" (at 200.66 124.46 0)
     (effects (font (size 1.27 1.27)) (justify left bottom))
   )
@@
     (effects (font (size 1.27 1.27)) (justify left bottom))
   )
-  (text "change values for\n0...825mV @VDD/4" (at 190.5 82.55 0)
+  (text "change values for\n0...825mV @VDD/4" (at 218.44 80.01 0)
     (effects (font (size 1.27 1.27)) (justify left bottom))
   )
@@
   )
   (text "adapt values" (at 152.4 50.8 0)
+    (effects (font (size 1.27 1.27)) (justify left bottom))
+  )
+  (text "tau = 1/(2*pi*f_{c}) = 1/(ω_{c})\nR*C = 100k*100n = 10ms -> 16Hz\nR*C = 100k*1u = 100ms -> 1.6Hz"
+    (at 243.84 105.41 0)
     (effects (font (size 1.27 1.27)) (justify left bottom))
   )
@@
     (effects (font (size 1.27 1.27)) (justify left bottom))
   )
-  (text "1.83...3.29V" (at 189.23 74.93 0)
+  (text "1.83...3.29V" (at 218.44 74.93 0)
     (effects (font (size 1.27 1.27)) (justify left bottom))
   )
@@
     (effects (font (size 1.27 1.27)) (justify left bottom))
   )
-  (text "change values for\n0...825mV @VDD/4" (at 189.23 138.43 0)
+  (text "change values for\n0...825mV @VDD/4" (at 217.17 137.16 0)
     (effects (font (size 1.27 1.27)) (justify left bottom))
   )
@@
     (effects (font (size 1.27 1.27)) (justify right))
   )
-  (hierarchical_label "BalaceCurrent" (shape output) (at 182.88 127 0)
+  (hierarchical_label "BalaceCurrent" (shape output) (at 194.31 127 0)
     (effects (font (size 1.27 1.27)) (justify left))
   )
-  (hierarchical_label "CellVoltage" (shape output) (at 182.88 71.12 0)
+  (hierarchical_label "CellVoltage" (shape output) (at 194.31 71.12 0)
     (effects (font (size 1.27 1.27)) (justify left))
   )
@@
     (pin "3")
   )
+  (symbol (lib_id "Device:C") (at 191.77 132.08 0) (unit 1)
+    (in_bom yes) (on_board yes) (fields_autoplaced)
+    (property "Reference" "C42" (id 0) (at 195.58 130.8099 0)
+      (effects (font (size 1.27 1.27)) (justify left))
+    )
+    (property "Value" "100n" (id 1) (at 195.58 133.3499 0)
+      (effects (font (size 1.27 1.27)) (justify left))
+    )
+    (property "Footprint" "Capacitor_SMD:C_0402_1005Metric" (id 2) (at 192.7352 135.89 0)
+      (effects (font (size 1.27 1.27)) hide)
+    )
+    (property "Datasheet" "~" (id 3) (at 191.77 132.08 0)
+      (effects (font (size 1.27 1.27)) hide)
+    )
+    (pin "1")
+    (pin "2")
+  )
   (symbol (lib_id "power:GND") (at 101.6 137.16 0) (unit 1)
     (in_bom yes) (on_board yes)
@@
     (property "Reference" "U9" (id 0) (at 165.1 111.3282 0))
     (property "Value" "TLV9052" (id 1) (at 165.1 113.6396 0))
-    (property "Footprint" "Package_SO:MSOP-8_3x3mm_P0.65mm" (id 2) (at 165.1 120.65 0)
+    (property "Footprint" "Package_TO_SOT_SMD:SOT-23-8" (id 2) (at 165.1 120.65 0)
       (effects (font (size 1.27 1.27)) hide)
     )
@@
     (pin "3")
   )
+  (symbol (lib_id "Device:C") (at 191.77 76.2 0) (unit 1)
+    (in_bom yes) (on_board yes) (fields_autoplaced)
+    (property "Reference" "C41" (id 0) (at 195.58 74.9299 0)
+      (effects (font (size 1.27 1.27)) (justify left))
+    )
+    (property "Value" "100n" (id 1) (at 195.58 77.4699 0)
+      (effects (font (size 1.27 1.27)) (justify left))
+    )
+    (property "Footprint" "Capacitor_SMD:C_0402_1005Metric" (id 2) (at 192.7352 80.01 0)
+      (effects (font (size 1.27 1.27)) hide)
+    )
+    (property "Datasheet" "~" (id 3) (at 191.77 76.2 0)
+      (effects (font (size 1.27 1.27)) hide)
+    )
+    (pin "1")
+    (pin "2")
+  )
   (symbol (lib_id "Device:R") (at 101.6 132.08 0) (unit 1)
     (in_bom yes) (on_board yes) (fields_autoplaced)
@@
     (pin "2")
   )
+  (symbol (lib_id "power:GND") (at 191.77 137.16 0) (unit 1)
+    (in_bom yes) (on_board yes)
+    (property "Reference" "#PWR037" (id 0) (at 191.77 143.51 0)
+      (effects (font (size 1.27 1.27)) hide)
+    )
+    (property "Value" "GND" (id 1) (at 191.897 141.5542 0)
+      (effects (font (size 1.27 1.27)) hide)
+    )
+    (property "Footprint" "" (id 2) (at 191.77 137.16 0)
+      (effects (font (size 1.27 1.27)) hide)
+    )
+    (property "Datasheet" "" (id 3) (at 191.77 137.16 0)
+      (effects (font (size 1.27 1.27)) hide)
+    )
+    (pin "1")
+  )
   (symbol (lib_id "Device:C") (at 134.62 62.23 0) (unit 1)
     (in_bom yes) (on_board yes) (fields_autoplaced)
@@
     (property "Reference" "U9" (id 0) (at 165.1 55.4482 0))
     (property "Value" "TLV9052" (id 1) (at 165.1 57.7596 0))
-    (property "Footprint" "Package_SO:MSOP-8_3x3mm_P0.65mm" (id 2) (at 165.1 64.77 0)
+    (property "Footprint" "Package_TO_SOT_SMD:SOT-23-8" (id 2) (at 165.1 64.77 0)
       (effects (font (size 1.27 1.27)) hide)
     )
@@
       (effects (font (size 1.27 1.27)) (justify left))
     )
-    (property "Footprint" "Package_SO:MSOP-8_3x3mm_P0.65mm" (id 2) (at 127 62.23 0)
+    (property "Footprint" "Package_TO_SOT_SMD:SOT-23-8" (id 2) (at 127 62.23 0)
       (effects (font (size 1.27 1.27)) hide)
     )
@@
     (pin "2")
   )
+  (symbol (lib_id "power:GND") (at 191.77 81.28 0) (unit 1)
+    (in_bom yes) (on_board yes)
+    (property "Reference" "#PWR030" (id 0) (at 191.77 87.63 0)
+      (effects (font (size 1.27 1.27)) hide)
+    )
+    (property "Value" "GND" (id 1) (at 191.897 85.6742 0)
+      (effects (font (size 1.27 1.27)) hide)
+    )
+    (property "Footprint" "" (id 2) (at 191.77 81.28 0)
+      (effects (font (size 1.27 1.27)) hide)
+    )
+    (property "Datasheet" "" (id 3) (at 191.77 81.28 0)
+      (effects (font (size 1.27 1.27)) hide)
+    )
+    (pin "1")
+  )
   (symbol (lib_id "power:GND") (at 181.61 81.28 0) (unit 1)

Commit message: Update
Parts:
- NT1: footprint (none) -> 0_ProjectLibrary:NetTie-2_SMD_Pad0.127mm
Connections:
- net Cell+: now also NT1.1; no longer R41.1
- net at NT1.2: now also R41.1
Other:
- moved on the sheet: NT1
Changed lines of the file:
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@@
   (junction (at 134.62 48.26) (diameter 0) (color 0 0 0 0)
   )
+  (junction (at 143.51 123.19) (diameter 0) (color 0 0 0 0)
+  )
   (junction (at 124.46 104.14) (diameter 0) (color 0 0 0 0)
   )
@@
   (junction (at 146.05 48.26) (diameter 0) (color 0 0 0 0)
   )
-  (junction (at 143.51 109.22) (diameter 0) (color 0 0 0 0)
-  )
   (junction (at 124.46 129.54) (diameter 0) (color 0 0 0 0)
   )
@@
   (junction (at 181.61 71.12) (diameter 0) (color 0 0 0 0)
   )
+  (junction (at 143.51 104.14) (diameter 0) (color 0 0 0 0)
+  )
   (junction (at 115.57 114.3) (diameter 0) (color 0 0 0 0)
   )
@@
   (junction (at 134.62 129.54) (diameter 0) (color 0 0 0 0)
   )
-  (junction (at 143.51 116.84) (diameter 0) (color 0 0 0 0)
-  )
   (wire (pts (xy 181.61 49.53) (xy 181.61 48.26))
     (stroke (width 0) (type default) (color 0 0 0 0))
@@
     (stroke (width 0) (type default) (color 0 0 0 0))
   )
-  (wire (pts (xy 148.59 123.19) (xy 157.48 123.19))
-    (stroke (width 0) (type default) (color 0 0 0 0))
-  )
   (wire (pts (xy 181.61 125.73) (xy 181.61 127))
     (stroke (width 0) (type default) (color 0 0 0 0))
@@
     (stroke (width 0) (type default) (color 0 0 0 0))
   )
+  (wire (pts (xy 143.51 123.19) (xy 157.48 123.19))
+    (stroke (width 0) (type default) (color 0 0 0 0))
+  )
   (wire (pts (xy 156.21 68.58) (xy 156.21 67.31))
     (stroke (width 0) (type default) (color 0 0 0 0))
@@
     (stroke (width 0) (type default) (color 0 0 0 0))
   )
-  (wire (pts (xy 148.59 109.22) (xy 148.59 104.14))
-    (stroke (width 0) (type default) (color 0 0 0 0))
-  )
   (wire (pts (xy 191.77 127) (xy 194.31 127))
     (stroke (width 0) (type default) (color 0 0 0 0))
@@
     (stroke (width 0) (type default) (color 0 0 0 0))
   )
-  (wire (pts (xy 148.59 116.84) (xy 148.59 123.19))
-    (stroke (width 0) (type default) (color 0 0 0 0))
-  )
   (wire (pts (xy 146.05 67.31) (xy 156.21 67.31))
     (stroke (width 0) (type default) (color 0 0 0 0))
@@
     (stroke (width 0) (type default) (color 0 0 0 0))
   )
-  (wire (pts (xy 143.51 116.84) (xy 148.59 116.84))
-    (stroke (width 0) (type default) (color 0 0 0 0))
-  )
   (wire (pts (xy 191.77 71.12) (xy 191.77 72.39))
     (stroke (width 0) (type default) (color 0 0 0 0))
@@
     (stroke (width 0) (type default) (color 0 0 0 0))
   )
-  (wire (pts (xy 148.59 104.14) (xy 181.61 104.14))
+  (wire (pts (xy 143.51 104.14) (xy 144.78 104.14))
     (stroke (width 0) (type default) (color 0 0 0 0))
   )
@@
     (stroke (width 0) (type default) (color 0 0 0 0))
   )
-  (wire (pts (xy 143.51 116.84) (xy 143.51 124.46))
+  (wire (pts (xy 143.51 116.84) (xy 143.51 123.19))
     (stroke (width 0) (type default) (color 0 0 0 0))
   )
@@
     (stroke (width 0) (type default) (color 0 0 0 0))
   )
-  (wire (pts (xy 143.51 109.22) (xy 148.59 109.22))
+  (wire (pts (xy 149.86 104.14) (xy 181.61 104.14))
     (stroke (width 0) (type default) (color 0 0 0 0))
   )
@@
     (stroke (width 0) (type default) (color 0 0 0 0))
   )
+  (wire (pts (xy 143.51 123.19) (xy 143.51 124.46))
+    (stroke (width 0) (type default) (color 0 0 0 0))
+  )
   (wire (pts (xy 181.61 135.89) (xy 181.61 137.16))
     (stroke (width 0) (type default) (color 0 0 0 0))
@@
     (effects (font (size 1.27 1.27)) (justify left bottom))
   )
-  (text "P = (1A)^2 * 0R1 = 0.1W\nPmax 0603 = 0.1...0.2W" (at 148.59 99.06 0)
+  (text "P = (1A)^2 * 0R1 = 0.1W\nPmax 0603 = 0.1...0.2W" (at 175.26 96.52 0)
     (effects (font (size 1.27 1.27)) (justify left bottom))
   )
@@
     (effects (font (size 1.27 1.27)) (justify right))
   )
-  (symbol (lib_id "Device:NetTie_2") (at 161.29 101.6 0) (unit 1)
-    (in_bom no) (on_board yes) (fields_autoplaced)
-    (property "Reference" "NT1" (id 0) (at 161.29 96.52 0))
-    (property "Value" "NetTie_2" (id 1) (at 161.29 99.06 0))
-    (property "Footprint" "" (id 2) (at 161.29 101.6 0)
+  (symbol (lib_id "Device:NetTie_2") (at 147.32 104.14 0) (unit 1)
+    (in_bom no) (on_board yes)
+    (property "Reference" "NT1" (id 0) (at 147.32 99.06 0))
+    (property "Value" "NetTie_2" (id 1) (at 147.32 101.6 0))
+    (property "Footprint" "0_ProjectLibrary:NetTie-2_SMD_Pad0.127mm" (id 2) (at 147.32 104.14 0)
       (effects (font (size 1.27 1.27)) hide)
     )
-    (property "Datasheet" "~" (id 3) (at 161.29 101.6 0)
+    (property "Datasheet" "~" (id 3) (at 147.32 104.14 0)
       (effects (font (size 1.27 1.27)) hide)
     )

Commit message: stream 24-01-24
Other:
- moved on the sheet: Q7, R30, R31, R32
Changed lines of the file:
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@@
   (junction (at 146.05 77.47) (diameter 0) (color 0 0 0 0)
   )
-  (junction (at 92.71 121.92) (diameter 0) (color 0 0 0 0)
+  (junction (at 92.71 149.86) (diameter 0) (color 0 0 0 0)
   )
   (junction (at 129.54 77.47) (diameter 0) (color 0 0 0 0)
@@
     (stroke (width 0) (type default) (color 0 0 0 0))
   )
-  (wire (pts (xy 92.71 121.92) (xy 91.44 121.92))
+  (wire (pts (xy 92.71 149.86) (xy 91.44 149.86))
     (stroke (width 0) (type default) (color 0 0 0 0))
   )
@@
     (stroke (width 0) (type default) (color 0 0 0 0))
   )
-  (wire (pts (xy 92.71 135.89) (xy 92.71 137.16))
+  (wire (pts (xy 92.71 163.83) (xy 92.71 165.1))
     (stroke (width 0) (type default) (color 0 0 0 0))
   )
@@
     (stroke (width 0) (type default) (color 0 0 0 0))
   )
-  (wire (pts (xy 101.6 114.3) (xy 101.6 116.84))
+  (wire (pts (xy 101.6 114.3) (xy 101.6 144.78))
     (stroke (width 0) (type default) (color 0 0 0 0))
   )
@@
     (stroke (width 0) (type default) (color 0 0 0 0))
   )
-  (wire (pts (xy 83.82 121.92) (xy 82.55 121.92))
-    (stroke (width 0) (type default) (color 0 0 0 0))
-  )
-  (wire (pts (xy 101.6 127) (xy 101.6 128.27))
+  (wire (pts (xy 83.82 149.86) (xy 82.55 149.86))
+    (stroke (width 0) (type default) (color 0 0 0 0))
+  )
+  (wire (pts (xy 101.6 154.94) (xy 101.6 156.21))
     (stroke (width 0) (type default) (color 0 0 0 0))
   )
@@
     (stroke (width 0) (type default) (color 0 0 0 0))
   )
-  (wire (pts (xy 101.6 135.89) (xy 101.6 137.16))
-    (stroke (width 0) (type default) (color 0 0 0 0))
-  )
-  (wire (pts (xy 93.98 121.92) (xy 92.71 121.92))
+  (wire (pts (xy 101.6 163.83) (xy 101.6 165.1))
+    (stroke (width 0) (type default) (color 0 0 0 0))
+  )
+  (wire (pts (xy 93.98 149.86) (xy 92.71 149.86))
     (stroke (width 0) (type default) (color 0 0 0 0))
   )
@@
     (stroke (width 0) (type default) (color 0 0 0 0))
   )
-  (wire (pts (xy 92.71 128.27) (xy 92.71 121.92))
+  (wire (pts (xy 92.71 156.21) (xy 92.71 149.86))
     (stroke (width 0) (type default) (color 0 0 0 0))
   )
@@
     (effects (font (size 1.27 1.27)) (justify left bottom))
   )
-  (hierarchical_label "BalanceControl" (shape input) (at 82.55 121.92 180)
+  (hierarchical_label "BalanceControl" (shape input) (at 82.55 149.86 180)
     (effects (font (size 1.27 1.27)) (justify right))
   )
@@
     (pin "2")
   )
-  (symbol (lib_id "power:GND") (at 101.6 137.16 0) (unit 1)
-    (in_bom yes) (on_board yes)
-    (property "Reference" "#PWR048" (id 0) (at 101.6 143.51 0)
-      (effects (font (size 1.27 1.27)) hide)
-    )
-    (property "Value" "GND" (id 1) (at 101.727 141.5542 0)
-      (effects (font (size 1.27 1.27)) hide)
-    )
-    (property "Footprint" "" (id 2) (at 101.6 137.16 0)
-      (effects (font (size 1.27 1.27)) hide)
-    )
-    (property "Datasheet" "" (id 3) (at 101.6 137.16 0)
+  (symbol (lib_id "power:GND") (at 101.6 165.1 0) (unit 1)
+    (in_bom yes) (on_board yes)
+    (property "Reference" "#PWR048" (id 0) (at 101.6 171.45 0)
+      (effects (font (size 1.27 1.27)) hide)
+    )
+    (property "Value" "GND" (id 1) (at 101.727 169.4942 0)
+      (effects (font (size 1.27 1.27)) hide)
+    )
+    (property "Footprint" "" (id 2) (at 101.6 165.1 0)
+      (effects (font (size 1.27 1.27)) hide)
+    )
+    (property "Datasheet" "" (id 3) (at 101.6 165.1 0)
       (effects (font (size 1.27 1.27)) hide)
     )
@@
     (pin "8")
   )
-  (symbol (lib_id "Device:Q_NMOS_GSD") (at 99.06 121.92 0) (unit 1)
-    (in_bom yes) (on_board yes)
-    (property "Reference" "Q7" (id 0) (at 104.2416 120.7516 0)
-      (effects (font (size 1.27 1.27)) (justify left))
-    )
-    (property "Value" "PMXB360ENEA" (id 1) (at 104.2416 123.063 0)
-      (effects (font (size 1.27 1.27)) (justify left))
-    )
-    (property "Footprint" "0_ProjectLibrary:DFN1010-3" (id 2) (at 104.14 119.38 0)
-      (effects (font (size 1.27 1.27)) hide)
-    )
-    (property "Datasheet" "~" (id 3) (at 99.06 121.92 0)
+  (symbol (lib_id "Device:Q_NMOS_GSD") (at 99.06 149.86 0) (unit 1)
+    (in_bom yes) (on_board yes)
+    (property "Reference" "Q7" (id 0) (at 104.2416 148.6916 0)
+      (effects (font (size 1.27 1.27)) (justify left))
+    )
+    (property "Value" "PMXB360ENEA" (id 1) (at 104.2416 151.003 0)
+      (effects (font (size 1.27 1.27)) (justify left))
+    )
+    (property "Footprint" "0_ProjectLibrary:DFN1010-3" (id 2) (at 104.14 147.32 0)
+      (effects (font (size 1.27 1.27)) hide)
+    )
+    (property "Datasheet" "~" (id 3) (at 99.06 149.86 0)
       (effects (font (size 1.27 1.27)) hide)
     )
@@
     (pin "2")
   )
-  (symbol (lib_id "Device:R") (at 101.6 132.08 0) (unit 1)
+  (symbol (lib_id "Device:R") (at 101.6 160.02 0) (unit 1)
     (in_bom yes) (on_board yes) (fields_autoplaced)
-    (property "Reference" "R32" (id 0) (at 99.06 130.8099 0)
+    (property "Reference" "R32" (id 0) (at 99.06 158.7499 0)
       (effects (font (size 1.27 1.27)) (justify right))
     )
-    (property "Value" "10k" (id 1) (at 99.06 133.3499 0)
+    (property "Value" "10k" (id 1) (at 99.06 161.2899 0)
       (effects (font (size 1.27 1.27)) (justify right))
     )
-    (property "Footprint" "Resistor_SMD:R_0402_1005Metric" (id 2) (at 99.822 132.08 90)
-      (effects (font (size 1.27 1.27)) hide)
-    )
-    (property "Datasheet" "~" (id 3) (at 101.6 132.08 0)
-      (effects (font (size 1.27 1.27)) hide)
-    )
-    (pin "1")
-    (pin "2")
-  )
-  (symbol (lib_id "Device:R") (at 92.71 132.08 0) (unit 1)
+    (property "Footprint" "Resistor_SMD:R_0402_1005Metric" (id 2) (at 99.822 160.02 90)
+      (effects (font (size 1.27 1.27)) hide)
+    )
+    (property "Datasheet" "~" (id 3) (at 101.6 160.02 0)
+      (effects (font (size 1.27 1.27)) hide)
+    )
+    (pin "1")
+    (pin "2")
+  )
+  (symbol (lib_id "Device:R") (at 92.71 160.02 0) (unit 1)
     (in_bom yes) (on_board yes) (fields_autoplaced)
-    (property "Reference" "R31" (id 0) (at 90.9574 130.9116 0)
+    (property "Reference" "R31" (id 0) (at 90.9574 158.8516 0)
       (effects (font (size 1.27 1.27)) (justify right))
     )
-    (property "Value" "100k" (id 1) (at 90.9574 133.223 0)
+    (property "Value" "100k" (id 1) (at 90.9574 161.163 0)
       (effects (font (size 1.27 1.27)) (justify right))
     )
-    (property "Footprint" "Resistor_SMD:R_0402_1005Metric" (id 2) (at 90.932 132.08 90)
-      (effects (font (size 1.27 1.27)) hide)
-    )
-    (property "Datasheet" "~" (id 3) (at 92.71 132.08 0)
+    (property "Footprint" "Resistor_SMD:R_0402_1005Metric" (id 2) (at 90.932 160.02 90)
+      (effects (font (size 1.27 1.27)) hide)
+    )
+    (property "Datasheet" "~" (id 3) (at 92.71 160.02 0)
       (effects (font (size 1.27 1.27)) hide)
     )
@@
     (pin "2")
   )
-  (symbol (lib_id "power:GND") (at 92.71 137.16 0) (unit 1)
-    (in_bom yes) (on_board yes)
-    (property "Reference" "#PWR047" (id 0) (at 92.71 143.51 0)
-      (effects (font (size 1.27 1.27)) hide)
-    )
-    (property "Value" "GND" (id 1) (at 92.837 141.5542 0)
-      (effects (font (size 1.27 1.27)) hide)
-    )
-    (property "Footprint" "" (id 2) (at 92.71 137.16 0)
-      (effects (font (size 1.27 1.27)) hide)
-    )
-    (property "Datasheet" "" (id 3) (at 92.71 137.16 0)
+  (symbol (lib_id "power:GND") (at 92.71 165.1 0) (unit 1)
+    (in_bom yes) (on_board yes)
+    (property "Reference" "#PWR047" (id 0) (at 92.71 171.45 0)
+      (effects (font (size 1.27 1.27)) hide)
+    )
+    (property "Value" "GND" (id 1) (at 92.837 169.4942 0)
+      (effects (font (size 1.27 1.27)) hide)
+    )
+    (property "Footprint" "" (id 2) (at 92.71 165.1 0)
+      (effects (font (size 1.27 1.27)) hide)
+    )
+    (property "Datasheet" "" (id 3) (at 92.71 165.1 0)
       (effects (font (size 1.27 1.27)) hide)
     )
@@
     (pin "8")
   )
-  (symbol (lib_id "Device:R") (at 87.63 121.92 270) (unit 1)
-    (in_bom yes) (on_board yes)
-    (property "Reference" "R30" (id 0) (at 87.63 124.841 90))
-    (property "Value" "1k" (id 1) (at 87.63 127.1524 90))
-    (property "Footprint" "Resistor_SMD:R_0402_1005Metric" (id 2) (at 87.63 120.142 90)
-      (effects (font (size 1.27 1.27)) hide)
-    )
-    (property "Datasheet" "~" (id 3) (at 87.63 121.92 0)
-      (effects (font (size 1.27 1.27)) hide)
-    )
+  (symbol (lib_id "Device:R") (at 87.63 149.86 270) (unit 1)
+    (in_bom yes) (on_board yes)
+    (property "Reference" "R30" (id 0) (at 87.63 152.781 90))
+    (property "Value" "1k" (id 1) (at 87.63 155.0924 90))
+    (property "Footprint" "Resistor_SMD:R_0402_1005Metric" (id 2) (at 87.63 148.082 90)
+      (effects (font (size 1.27 1.27)) hide)
+    )
+    (property "Datasheet" "~" (id 3) (at 87.63 149.86 0)
+      (effects (font (size 1.27 1.27)) hide)
+    )

Commit message: finishing touches in preparation for manufacturing
Parts:
- added TP24: PWM, 0_ProjectLibrary:TestPoint_Pad_D1.0mm, symbol Connector:TestPoint
- added TP25: Voltage, 0_ProjectLibrary:TestPoint_Pad_D1.0mm, symbol Connector:TestPoint
- added TP26: Current, 0_ProjectLibrary:TestPoint_Pad_D1.0mm, symbol Connector:TestPoint
- renumbered C15 to C44, C16 to C45, C17 to C46, C41 to C47, C42 to C48, NT1 to NT8, Q7 to Q36, Q8 to Q37, Q9 to Q38, Q10 to Q39, Q11 to Q40, R33 to R100, R34 to R101, R35 to R102, R36 to R103, R37 to R104, R38 to R105, R39 to R106, R40 to R107, R41 to R108, R42 to R109, R30 to R97, R31 to R98, R32 to R99, U9 to U12
Connections:
- net BalaceCurrent: now also TP26.1
- net CellVoltage: now also TP25.1
- net at Q36.3 (D), Q37.1 (B), R100.2: now also TP24.1
Other:
- note removed: "PWM"
- title: (none) -> 8-Cell Balancer
