File: Blancer1-8.kicad_sch (KiCad schematic)
At the start: 28 parts, among them Q36 PMXB360ENEA, Q37 2SA1832, Q38 IRLU120NPBF, Q39 BSS84AKW, Q40 BSS84AKW, U12 TLV9052

Commit message: finalize component values
Parts:
- NT8: value NetTie_2 -> NetTie
- R100, R99: value 10k -> 22k
- R101: value 10k -> 47k
- R104, R106: value 100k -> 4.7k
- R105: value 270k -> 22k
- R107: value 270k -> 4.7k
- R108: value 10k -> 620R
- R109: value 330k -> 4.7k
- R97: value 1k -> 620R
Other:
- note added: "0.1R * 4.7k / 620R = 0.758 I_{bal,max} = 0.825V / 0.758 = 1.09A"
- note added: "0.44~0.79V"
- note added: "0.44~0.79V max. 0.825V @VDD/4"
- note added: "0~0.1V"
- note added: "0~0.76V max. 0.825V @VDD/4"
- note added: "30uA"
- note added: "4.7k / (4.7k + 22k) * 4.7k / 4.7k = 0.176 V_{Cell,max} = 0.825V / 0.176 = 4.69V"
- note added: "420Hz"
- note added: "I_{leakage,max} = 1uA"
- note added: "Ibal = 0~1A Vcm = 3.1~4.4V @ 1A"
- note added: "P_{FET,max} = 32V * 168uA = 5.4mW"
- note added: "P_{FET,max} = 35V * 80uA = 2.8mW"
- note added: "P_{Shunt} = (1A)^2 * 0.1R = 0.1W P_{0603,max} = 0.1~0.2W"
- note added: "Vcell = 2.5~4.5V Vcm = 2.06~3.71V"
- note added: "Vgs = 0~3.1V TO251 (IPAK) 1.5A @ 2.5V"
- note added: "Vgs margin to rail -2.06~-3.71V @ 94~168uA"
- note added: "Vgs margin to rail -3.1~-4.4V @ 161uA"
- note added: "max 90uA"
- note added: "~80uA"
- note removed: "0...0.1V"
- note removed: "0.68...1.22V"
- note removed: "1.5A @ 2.5V"
- note removed: "1.83...3.29V"
- note removed: "100...200uA"
- note removed: "100k / (100k + 270k) * 270k / 100k = 0.730 3.3V / 0.730 = 4.52V"
- note removed: "22Hz"
- note removed: "70uA"
- note removed: "I_{leakage} = 1uA"
- note removed: "Ibal = 0...1A"
- note removed: "P = (1A)^2 * 0R1 = 0.1W Pmax 0603 = 0.1...0.2W"
- note removed: "Pmax = 32V * 12.2uA = 390uW"
- note removed: "Pmax = 33V * 10uA = 330uW"
- note removed: "TO251 (IPAK)"
- note removed: "Vcell = 2.5...4.5V"
- note removed: "Vcm = 1.83...3.29V"
- note removed: "Vcm = 3.1...4.4V @ 1A"
- note removed: "Vgs = 0...3.2V"
- note removed: "Vgs margin to rail -1.83...-3.29V @ 6.8...12.2uA"
- note removed: "Vgs margin to rail -3.1...-4.4V @ 10uA"
- note removed: "adapt values"
- note removed: "change values for 0...825mV @VDD/4"
- note removed: "max. 500uA"
- note removed: "tau = 1/(2*pi*f_{c}) = 1/(ω_{c}) R*C = 100k*100n = 10ms -> 16Hz R*C = 100k*1u = 100ms -> 1.6Hz"
- moved on the sheet: C44, C45, C46, C47, C48, NT8, Q36, Q37, Q38, Q39, Q40, R100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
