File: Hardware/8-Cell Balancer.kicad_pcb (KiCad board)
At the start: 2 copper layers, 60 x 50 mm, 251 parts, among them J1 Balance, J2 Conn_01x06, Q1 PMXB360ENEA, Q10 BSS84AKW, Q11 PMXB360ENEA, Q12 2SA1832, Q13 IRLU120NPBF, Q14 BSS84AKW, Q15 BSS84AKW, Q16 PMXB360ENEA, Q17 2SA1832, Q18 IRLU120NPBF, Q19 BSS84AKW, Q2 2SA1832, Q20 BSS84AKW, Q21 PMXB360ENEA, Q22 2SA1832, Q23 IRLU120NPBF, Q24 BSS84AKW, Q25 BSS84AKW, Q26 PMXB360ENEA, Q27 2SA1832, Q28 IRLU120NPBF, Q29 BSS84AKW, Q3 IRLU120NPBF, Q30 BSS84AKW, Q31 PMXB360ENEA, Q32 2SA1832, Q33 IRLU120NPBF, Q34 BSS84AKW, Q35 BSS84AKW, Q36 PMXB360ENEA, Q37 2SA1832, Q38 IRLU120NPBF, Q39 BSS84AKW, Q4 BSS84AKW, Q40 BSS84AKW, Q5 BSS84AKW, Q6 PMXB360ENEA, Q7 2SA1832, Q8 IRLU120NPBF, Q9 BSS84AKW, SW1 Reset, SW2 Button, U1 AP7370, U10 TLV9052, U11 TLV9052, U12 TLV9052, U2 74HC4051, U3 74HC4051, U4 NINA-B306, U5 TLV9052, U6 TLV9052, U7 TLV9052, U8 TLV9052, U9 TLV9052

Commit message: generate BOM
Parts:
- C11, C16, C21, C26, C31, C36, C41, C46: value 100n -> DNP
- J2: value Conn_01x06 -> SWD
- NT1, NT2, NT3, NT4, NT5, NT6, NT7, NT8: value NetTie_2 -> NetTie
- R1, R2: value 51k -> 47k
- R10, R101, R23, R36, R49, R62, R75, R88: value 10k -> 47k
- R100, R21, R22, R34, R35, R47, R48, R60, R61, R73, R74, R8, R86, R87, R9, R99: value 10k -> 22k
- R104, R106, R13, R15, R26, R28, R39, R41, R52, R54, R65, R67, R78, R80, R91, R93: value 100k -> 4.7k
- R105, R14, R27, R40, R53, R66, R79, R92: value 270k -> 22k
- R107, R16, R29, R42, R55, R68, R81, R94: value 270k -> 4.7k
- R108, R17, R30, R43, R56, R69, R82, R95: value 10k -> 620R
- R109, R18, R31, R44, R57, R70, R83, R96: value 330k -> 4.7k
- R19, R32, R45, R58, R6, R71, R84, R97: value 1k -> 620R
- R3, R4, R5: value 1.8k -> 620R

Commit message: hardware: version 1
Parts:
- removed Q1, Q11, Q16, Q21, Q26, Q31, Q36, Q6: PMXB360ENEA, 0_ProjectLibrary:DFN1010-3
- removed Q12, Q17, Q2, Q22, Q27, Q32, Q37, Q7: 2SA1832, Package_TO_SOT_SMD:SOT-416
- removed R10, R101, R23, R36, R49, R62, R75, R88: 47k, Resistor_SMD:R_0402_1005Metric
- removed R100, R21, R22, R34, R35, R47, R48, R60, R61, R73, R74, R8, R86, R87, R9, R99: 22k, Resistor_SMD:R_0402_1005Metric
- removed R19, R32, R45, R58, R6, R71, R84, R97: 620R, Resistor_SMD:R_0402_1005Metric
- removed R20, R33, R46, R59, R7, R72, R85, R98: 100k, Resistor_SMD:R_0402_1005Metric
- added C49: 3.3n, Capacitor_SMD:C_0402_1005Metric, F.Cu at (-24.5, 15.0)
- added C50: 3.3n, Capacitor_SMD:C_0402_1005Metric, F.Cu at (-23.5, 15.0)
- added C51: 3.3n, Capacitor_SMD:C_0402_1005Metric, F.Cu at (-22.5, 15.0)
- added C52: 3.3n, Capacitor_SMD:C_0402_1005Metric, F.Cu at (-21.5, 15.0)
- added C53: 3.3n, Capacitor_SMD:C_0402_1005Metric, F.Cu at (-21.5, -15.0)
- added C54: 3.3n, Capacitor_SMD:C_0402_1005Metric, F.Cu at (-22.5, -15.0)
- added C55: 3.3n, Capacitor_SMD:C_0402_1005Metric, F.Cu at (-23.5, -15.0)
- added C56: 3.3n, Capacitor_SMD:C_0402_1005Metric, F.Cu at (-24.5, -15.0)
- added D10: RB751S40, Diode_SMD:D_SOD-523, F.Cu at (17.0, 22.7)
- added D11: RB751S40, Diode_SMD:D_SOD-523, F.Cu at (9.00, 22.7)
- added D12: RB751S40, Diode_SMD:D_SOD-523, F.Cu at (1.00, 22.7)
- added D13: RB751S40, Diode_SMD:D_SOD-523, F.Cu at (-7.00, 22.7)
- added D14: RB751S40, Diode_SMD:D_SOD-523, F.Cu at (-2.00, -22.7)
- added D15: RB751S40, Diode_SMD:D_SOD-523, F.Cu at (6.00, -22.7)
- added D16: RB751S40, Diode_SMD:D_SOD-523, F.Cu at (14.0, -22.7)
- added D17: RB751S40, Diode_SMD:D_SOD-523, F.Cu at (22.0, -22.7)
- added D18: RB751S40, Diode_SMD:D_SOD-523, F.Cu at (22.0, 22.7)
- added D19: RB751S40, Diode_SMD:D_SOD-523, F.Cu at (14.0, 22.7)
- added D2: BZT52H-C6V2, Diode_SMD:D_SOD-123F, F.Cu at (21.2, 4.40)
- added D20: RB751S40, Diode_SMD:D_SOD-523, F.Cu at (6.00, 22.7)
- added D21: RB751S40, Diode_SMD:D_SOD-523, F.Cu at (-2.00, 22.7)
- added D22: RB751S40, Diode_SMD:D_SOD-523, F.Cu at (-7.00, -22.7)
- added D23: RB751S40, Diode_SMD:D_SOD-523, F.Cu at (1.00, -22.7)
- added D24: RB751S40, Diode_SMD:D_SOD-523, F.Cu at (9.00, -22.7)
- added D25: RB751S40, Diode_SMD:D_SOD-523, F.Cu at (17.0, -22.7)
- added D26: RB751S40, Diode_SMD:D_SOD-523, F.Cu at (19.5, 20.6)
- added D27: RB751S40, Diode_SMD:D_SOD-523, F.Cu at (11.5, 20.6)
- added D28: RB751S40, Diode_SMD:D_SOD-523, F.Cu at (3.50, 20.6)
- added D29: RB751S40, Diode_SMD:D_SOD-523, F.Cu at (-4.50, 20.6)
- added D3: BZT52H-C6V2, Diode_SMD:D_SOD-123F, F.Cu at (13.2, 4.40)
- added D30: RB751S40, Diode_SMD:D_SOD-523, F.Cu at (-4.50, -20.6)
- added D31: RB751S40, Diode_SMD:D_SOD-523, F.Cu at (3.50, -20.6)
- added D32: RB751S40, Diode_SMD:D_SOD-523, F.Cu at (11.5, -20.6)
- added D33: RB751S40, Diode_SMD:D_SOD-523, F.Cu at (19.5, -20.6)
- added D4: BZT52H-C6V2, Diode_SMD:D_SOD-123F, F.Cu at (5.20, 4.40)
- added D5: BZT52H-C6V2, Diode_SMD:D_SOD-123F, F.Cu at (-2.80, 4.40)
- added D6: BZT52H-C6V2, Diode_SMD:D_SOD-123F, F.Cu at (-6.20, -4.40)
- added D7: BZT52H-C6V2, Diode_SMD:D_SOD-123F, F.Cu at (1.80, -4.40)
- added D8: BZT52H-C6V2, Diode_SMD:D_SOD-123F, F.Cu at (9.80, -4.40)
- added D9: BZT52H-C6V2, Diode_SMD:D_SOD-123F, F.Cu at (17.8, -4.40)
- added FID1: Fiducial, Fiducial:Fiducial_1mm_Mask2mm, F.Cu at (-24.0, -23.0)
- added FID2: Fiducial, Fiducial:Fiducial_1mm_Mask2mm, F.Cu at (28.0, -23.0)
- added FID3: Fiducial, Fiducial:Fiducial_1mm_Mask2mm, F.Cu at (28.0, 23.0)
- added FID4: Fiducial, Fiducial:Fiducial_1mm_Mask2mm, F.Cu at (-24.0, 23.0)
- added R118: 620R, Resistor_SMD:R_0402_1005Metric, F.Cu at (16.6, 15.8)
- added R119: 620R, Resistor_SMD:R_0402_1005Metric, F.Cu at (8.60, 15.8)
- added R120: 620R, Resistor_SMD:R_0402_1005Metric, F.Cu at (0.60, 15.8)
- added R121: 620R, Resistor_SMD:R_0402_1005Metric, F.Cu at (-7.40, 15.8)
- added R122: 620R, Resistor_SMD:R_0402_1005Metric, F.Cu at (-1.60, -15.8)
- added R123: 620R, Resistor_SMD:R_0402_1005Metric, F.Cu at (6.40, -15.8)
- added R124: 620R, Resistor_SMD:R_0402_1005Metric, F.Cu at (14.4, -15.8)
- added R125: 620R, Resistor_SMD:R_0402_1005Metric, F.Cu at (22.4, -15.8)
- added R126: 22k, Resistor_SMD:R_0402_1005Metric, F.Cu at (19.0, 22.3)
- added R127: 22k, Resistor_SMD:R_0402_1005Metric, F.Cu at (11.0, 22.3)
- added R128: 22k, Resistor_SMD:R_0402_1005Metric, F.Cu at (3.00, 22.3)
- added R129: 22k, Resistor_SMD:R_0402_1005Metric, F.Cu at (-5.00, 22.3)
- added R130: 22k, Resistor_SMD:R_0402_1005Metric, F.Cu at (-4.00, -22.3)
- added R131: 22k, Resistor_SMD:R_0402_1005Metric, F.Cu at (4.00, -22.3)
- added R132: 22k, Resistor_SMD:R_0402_1005Metric, F.Cu at (12.0, -22.3)
- added R133: 22k, Resistor_SMD:R_0402_1005Metric, F.Cu at (20.0, -22.3)
- added R134: 620R, Resistor_SMD:R_0402_1005Metric, F.Cu at (20.0, 22.3)
- added R135: 620R, Resistor_SMD:R_0402_1005Metric, F.Cu at (12.0, 22.3)
- added R136: 620R, Resistor_SMD:R_0402_1005Metric, F.Cu at (4.00, 22.3)
- added R137: 620R, Resistor_SMD:R_0402_1005Metric, F.Cu at (-4.00, 22.3)
- added R138: 620R, Resistor_SMD:R_0402_1005Metric, F.Cu at (-5.00, -22.3)
- added R139: 620R, Resistor_SMD:R_0402_1005Metric, F.Cu at (3.00, -22.3)
- added R140: 620R, Resistor_SMD:R_0402_1005Metric, F.Cu at (11.0, -22.3)
- added R141: 620R, Resistor_SMD:R_0402_1005Metric, F.Cu at (19.0, -22.3)
- C1, C2: footprint Capacitor_SMD:C_0402_1005Metric -> Capacitor_SMD:C_0603_1608Metric
- C11, C16, C21, C26, C31, C36, C41, C46: value DNP -> 100n
- R1, R2: value 47k -> 22k
- R102, R11, R24, R37, R50, R63, R76, R89: value 100k -> 330k
- SW1: value Reset -> B3U-1000
- SW2: value Button -> B3U-1000
- moved C1 5.20 mm to (-9.40, -14.2)
- moved TP12 5.14 mm to (-21.5, 16.6)
- moved TP15 5.14 mm to (-21.5, -16.6)
- moved TP18 5.06 mm to (-22.5, -16.6)
- moved TP9 5.06 mm to (-22.5, 16.6)
- moved TP21 5.02 mm to (-23.5, -16.6)
- moved TP6 5.02 mm to (-23.5, 16.6)
- moved TP24 5.00 mm to (-24.5, -16.6)
- moved TP3 5.00 mm to (-24.5, 16.6)
- moved U1 5.00 mm to (-11.5, -14.2)
- moved C2 4.80 mm to (-13.6, -14.2)
- moved R102 3.28 mm to (22.5, -18.5)
- moved R11 3.28 mm to (16.5, 18.5)
- moved R24 3.28 mm to (8.50, 18.5)
- moved R37 3.28 mm to (0.50, 18.5)
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Connections:
- C11 pad 1: Net-(C11-Pad1) -> /Balancer1/Cell+
- C11 pad 2: GND -> Net-(U5A-+)
- C16 pad 1: Net-(C16-Pad1) -> /Balancer2/Cell+
- C16 pad 2: /Balancer1/Cell+ -> Net-(U6A-+)
- C21 pad 1: Net-(C21-Pad1) -> /Balancer3/Cell+
- C21 pad 2: /Balancer2/Cell+ -> Net-(U7A-+)
- C26 pad 1: Net-(C26-Pad1) -> /Supply
- C26 pad 2: /Balancer3/Cell+ -> Net-(U8A-+)
- C31 pad 1: Net-(C31-Pad1) -> /Balancer5/Cell+
- C31 pad 2: /Supply -> Net-(U9A-+)
- C36 pad 1: Net-(C36-Pad1) -> /Balancer6/Cell+
- C36 pad 2: /Balancer5/Cell+ -> Net-(U10A-+)
- C41 pad 1: Net-(C41-Pad1) -> /Balancer7/Cell+
- C41 pad 2: /Balancer6/Cell+ -> Net-(U11A-+)
- C46 pad 1: Net-(C46-Pad1) -> /Balancer8/Cell+
- C46 pad 2: /Balancer7/Cell+ -> Net-(U12A-+)
- J2 pad 5: /TX -> /RX
- J2 pad 6: /RX -> /TX
- Q13 pad 2: Net-(Q13-Pad2) -> Net-(Q13-D)
- Q18 pad 2: Net-(Q18-Pad2) -> Net-(Q18-D)
- Q23 pad 2: Net-(Q23-Pad2) -> Net-(Q23-D)
- Q28 pad 2: Net-(Q28-Pad2) -> Net-(Q28-D)
- Q3 pad 2: Net-(Q3-Pad2) -> Net-(Q3-D)
- Q33 pad 2: Net-(Q33-Pad2) -> Net-(Q33-D)
- Q38 pad 2: Net-(Q38-Pad2) -> Net-(Q38-D)
- Q8 pad 2: Net-(Q8-Pad2) -> Net-(Q8-D)
- R103 pad 2: Net-(Q38-Pad2) -> Net-(Q38-D)
- R104 pad 1: Net-(C46-Pad1) -> Net-(U12A-+)
- R105 pad 1: Net-(C46-Pad1) -> Net-(U12A-+)
- R12 pad 2: Net-(Q3-Pad2) -> Net-(Q3-D)
- R13 pad 1: Net-(C11-Pad1) -> Net-(U5A-+)
- R14 pad 1: Net-(C11-Pad1) -> Net-(U5A-+)
- R25 pad 2: Net-(Q8-Pad2) -> Net-(Q8-D)
- R26 pad 1: Net-(C16-Pad1) -> Net-(U6A-+)
- R27 pad 1: Net-(C16-Pad1) -> Net-(U6A-+)
- R38 pad 2: Net-(Q13-Pad2) -> Net-(Q13-D)
- R39 pad 1: Net-(C21-Pad1) -> Net-(U7A-+)
- R40 pad 1: Net-(C21-Pad1) -> Net-(U7A-+)
- R51 pad 2: Net-(Q18-Pad2) -> Net-(Q18-D)
- R52 pad 1: Net-(C26-Pad1) -> Net-(U8A-+)
- R53 pad 1: Net-(C26-Pad1) -> Net-(U8A-+)
- R64 pad 2: Net-(Q23-Pad2) -> Net-(Q23-D)
- R65 pad 1: Net-(C31-Pad1) -> Net-(U9A-+)
- R66 pad 1: Net-(C31-Pad1) -> Net-(U9A-+)
- R77 pad 2: Net-(Q28-Pad2) -> Net-(Q28-D)
- R78 pad 1: Net-(C36-Pad1) -> Net-(U10A-+)
- R79 pad 1: Net-(C36-Pad1) -> Net-(U10A-+)
- R90 pad 2: Net-(Q33-Pad2) -> Net-(Q33-D)
- R91 pad 1: Net-(C41-Pad1) -> Net-(U11A-+)
- R92 pad 1: Net-(C41-Pad1) -> Net-(U11A-+)
- U10 pad 3: Net-(C36-Pad1) -> Net-(U10A-+)
- U10 pad 5: Net-(Q28-Pad2) -> Net-(U10B-+)
- U11 pad 3: Net-(C41-Pad1) -> Net-(U11A-+)
- U11 pad 5: Net-(Q33-Pad2) -> Net-(U11B-+)
- U12 pad 3: Net-(C46-Pad1) -> Net-(U12A-+)
- U12 pad 5: Net-(Q38-Pad2) -> Net-(U12B-+)
- U5 pad 3: Net-(C11-Pad1) -> Net-(U5A-+)
- U5 pad 5: Net-(Q3-Pad2) -> Net-(U5B-+)
- U6 pad 3: Net-(C16-Pad1) -> Net-(U6A-+)
- U6 pad 5: Net-(Q8-Pad2) -> Net-(U6B-+)
- U7 pad 3: Net-(C21-Pad1) -> Net-(U7A-+)
- U7 pad 5: Net-(Q13-Pad2) -> Net-(U7B-+)
- U8 pad 3: Net-(C26-Pad1) -> Net-(U8A-+)
- U8 pad 5: Net-(Q18-Pad2) -> Net-(U8B-+)
- U9 pad 3: Net-(C31-Pad1) -> Net-(U9A-+)
- U9 pad 5: Net-(Q23-Pad2) -> Net-(U9B-+)
Routing:
- net Net-(Q8-D): track 0.00 -> 16.3 mm
- net Net-(Q33-D): track 0.00 -> 16.3 mm
- net Net-(Q28-D): track 0.00 -> 16.3 mm
- net Net-(Q23-D): track 0.00 -> 16.3 mm
- net Net-(Q18-D): track 0.00 -> 16.3 mm
- net Net-(Q13-D): track 0.00 -> 16.3 mm
- net Net-(Q38-D): track 0.00 -> 16.3 mm
- net Net-(Q3-D): track 0.00 -> 16.3 mm
- net Net-(Q33-Pad2): track 15.3 -> 0.00 mm
- net Net-(Q8-Pad2): track 15.3 -> 0.00 mm
- net Net-(Q38-Pad2): track 15.3 -> 0.00 mm
- net Net-(Q18-Pad2): track 15.3 -> 0.00 mm
- net Net-(Q13-Pad2): track 15.3 -> 0.00 mm
- net Net-(Q3-Pad2): track 15.3 -> 0.00 mm
- net Net-(Q28-Pad2): track 15.3 -> 0.00 mm
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Other:
- board text added: "1"
- board text added: "2"
- board text added: "3"
- board text added: "4"
- board text added: "5"
- board text added: "6"
- board text added: "7"
- board text added: "8"
- board text added: "8-Cell Balancer V1 by jbussmann"
- board text added: "IO CL RS GD RX TX"
- board text removed: "4 3 2 1"
- board text removed: "5 6 7 8"
- board text removed: "8-Cell Balancer by jbussmann"
- board text removed: "IO CL RS GD TX RX"
